File: TRECRCP.kicad_sch (KiCad schematic)
At the start: 47 parts, among them K1 12v Coil Relay, K2 12v Coil Relay, K5 Fujitsu_FTR-LYCA005x, K6 Fujitsu_FTR-LYCA005x, K7 Fujitsu_FTR-LYCA005x, Q2 IRLZ44NPBF, Q3 IRLZ44NPBF, Q4 IRLZ44NPBF, SW1 Dispatch2, SW1 Maint/Off/On Switch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

Commit message: Final Drive System
Removed VClamp, LED relays, and updated EStop circuit
Parts:
- removed D2, D3, D4: 1N4007, Diode_THT:D_DO-41_SOD81_P10.16mm_Horizontal, symbol Diode:1N4007
- removed D5, D6: LED, symbol Device:LED
- removed K5, K6, K7: Fujitsu_FTR-LYCA005x, Relay_THT:Relay_SPDT_Fujitsu_FTR-LYCA005x_FormC_Vertical, symbol Relay:Fujitsu_FTR-LYCA005x
- removed LL_Mosfet, LL_Mosfet1: P-Channel, Package_TO_SOT_SMD:SOT-23, symbol Transistor_FET:2N7002H
- removed Q2, Q3, Q4: IRLZ44NPBF, Package_TO_SOT_SMD:SOT-23, symbol Transistor_FET:2N7002H
- removed R1, R2: R220, symbol Device:R
- removed R3: R1k, symbol Device:R
- removed U5: RoboClaw VClamp, symbol CustomSymbols:RoboclawVClamp
- removed U6: Clamp Resistor, symbol CustomSymbols:Power_Resistor
- added D8, D9: LED, symbol Device:LED
- added LL_Mosfet2, LL_Mosfet3: IRLZ34N, Package_TO_SOT_SMD:SOT-23, symbol Transistor_FET:2N7002H
- added R4, R5: R220, symbol Device:R
- added R4, R5: R1K, symbol Device:R
Connections:
- net +5V: no longer Tower_A.3 (VCC), U1. (5VDC)
- net 120V: no longer K2.14
- net E-Stop Button: now also LL_Mosfet2.2 (S)
- net E-Stop Signal Out: now also LL_Mosfet3.3 (D)
- net GND: now also D8.1 (K), D9.1 (K), R4.1, R5.1
- net NEUT: no longer SW1.3 (K), SW4.3 (K), SW8.3 (K)
- net PLC E-Stop Trigger: now also LL_Mosfet2.1 (G), R4.2, R4.2
- net RCC E-Stop Trigger: now also LL_Mosfet3.1 (G), R5.2, R5.2
- net at SW5.3 (K): no longer SW1.4 (A)
- net at RCC1. (USB-C): now also U2.3 (USB-C); no longer U3. (Micro_USB)
- net +24V renamed 24V
- net Dispatch LED Power (120VAC): no longer names the net of SW5.4 (A)
- net Reset LED Power (120VAC): no longer names the net of SW4.4 (A)
- net Stop LED Power (120VAC): no longer names the net of SW8.4 (A)
- new net: D9.2 (A), R5.1
- new net: LL_Mosfet2.3 (D), LL_Mosfet3.2 (S)
- new net: D8.2 (A), R4.1
- new net: RCC1. (USB-C), U3. (Micro_USB)
- new net: Tower_A.3 (VCC), U1. (5VDC)
Other:
- note removed: "PUSHBUTTON LED DRIVER"
